File: Berrydock Mini/berrydock-mini.sch (KiCad schematic (older format))
At the start: 95 parts, among them J1 RJ45, P1 CONN_01X16, P2 CONN_01X16, P3 CONN_01X04, P4 CONN_01X03, P5 USB_OTG, P6 USB_A, SW1 SWITCH_INV, SW2 BUTTON, U1 USBLC6-2, U10 L6920DC, U11 FS8205A, U12 DW01-P, U13 USBLC6-2, U14 USBLC6-2, U15 CP2102, U2 USBLC6-2, U3 TD6811, U4 H1260NL, U5 Omega2, U6 SMP75, U7 SMP75, U8 ACT4088, U9 MCP73831

Commit message: First part of layout done
Parts:
- removed P2: CONN_01X16, Pin_Headers:Pin_Header_Straight_1x16, symbol CONN_01X16
- removed R22: 1K, Resistors_SMD:R_0603_HandSoldering, symbol R_Small
- added P2: CONN_01X11, Pin_Headers:Pin_Header_Straight_1x11, symbol CONN_01X11
Connections:
- net +3.3VP: now also P2.6 (P6)
- net +3V3: now also P2.2 (P2)
- net +5V: now also P2.11 (P11)
- net FW_RST: now also P2.5 (P5)
- net GND: now also P2.1 (P1)
- net GPIO18: now also P2.7 (P7)
- net GPIO19: now also P2.8 (P8)
- net GPIO4: now also P2.9 (P9)
- net GPIO5: now also P2.10 (P10)
- net RX0: now also P2.3 (P3)
- net TX0: now also P2.4 (P4)
Changed lines of the file:
@@
-$EndComp
-$Comp
-L R_Small R22
-U 1 1 57E96C09
-P 9100 6600
-F 0 "R22" H 9130 6620 50  0000 L CNN
-F 1 "1K" H 9130 6560 50  0000 L CNN
-F 2 "Resistors_SMD:R_0603_HandSoldering" H 9100 6600 50  0001 C CNN
-F 3 "" H 9100 6600 50  0000 C CNN
-	1    9100 6600
-	0    -1   -1   0
 $EndComp
 $Comp
@@
 F 0 "SW1" H 2150 1650 50  0000 C CNN
 F 1 "SWITCH_INV" H 2200 1350 50  0000 C CNN
-F 2 "Omega2-Berrydock:SMD-SLIDESWITCH" H 2350 1500 50  0000 C CNN
+F 2 "Omega2-Berrydock:SMD-SLIDESWITCH" H 2350 1500 50  0001 C CNN
 F 3 "" H 2350 1500 50  0000 C CNN
 	1    2350 1500
@@
 F 0 "SW2" H 11530 6410 50  0000 C CNN
 F 1 "BUTTON" H 11500 6250 50  0000 C CNN
-F 2 "Omega2-Berrydock:SMD-BUTTON-2x4x3,5" H 11450 6500 50  0000 C CNN
+F 2 "Omega2-Berrydock:SMD-BUTTON-2x4x3,5" H 11450 6500 50  0001 C CNN
 F 3 "" H 11450 6500 50  0000 C CNN
 	1    11450 6300
@@
 L +3.3VP #PWR069
 U 1 1 57EA972F
-P 2400 5950
-F 0 "#PWR069" H 2550 5900 50  0001 C CNN
-F 1 "+3.3VP" H 2400 6050 50  0000 C CNN
-F 2 "" H 2400 5950 50  0000 C CNN
-F 3 "" H 2400 5950 50  0000 C CNN
-	1    2400 5950
-	1    0    0    -1
-$EndComp
-Wire Wire Line
-	2400 5950 2400 6050
-Wire Wire Line
-	2400 6050 1900 6050
+P 2400 5750
+F 0 "#PWR069" H 2550 5700 50  0001 C CNN
+F 1 "+3.3VP" H 2400 5850 50  0000 C CNN
+F 2 "" H 2400 5750 50  0000 C CNN
+F 3 "" H 2400 5750 50  0000 C CNN
+	1    2400 5750
+	1    0    0    -1
+$EndComp
+Wire Wire Line
+	2400 5750 2400 5850
+Wire Wire Line
+	2400 5850 1900 5850
 $Comp
 L +3.3V #PWR070
@@
 Wire Wire Line
 	2300 5450 1900 5450
+Text Label 2200 5550 2    39   ~ 0
+RX0
+Text Label 2200 5650 2    39   ~ 0
+TX0
+Text Label 2200 5750 2    39   ~ 0
+FW_RST
+Text Label 2200 5950 2    39   ~ 0
+GPIO18
+Text Label 2200 6050 2    39   ~ 0
+GPIO19
 Text Label 2200 6150 2    39   ~ 0
-ETH_TX-
+GPIO4
 Text Label 2200 6250 2    39   ~ 0
-ETH_TX+
-Text Label 2200 6350 2    39   ~ 0
-ETH_RX-
-Text Label 2200 6450 2    39   ~ 0
-ETH_RX+
-Wire Wire Line
-	2200 6150 1900 6150
-Wire Wire Line
-	1900 6250 2200 6250
-Wire Wire Line
-	2200 6350 1900 6350
-Wire Wire Line
-	1900 6450 2200 6450
-Text Label 2200 5650 2    39   ~ 0
-UH_-
-Text Label 2200 5550 2    39   ~ 0
-UH_+
-Text Label 2200 5750 2    39   ~ 0
-RX0
-Text Label 2200 5850 2    39   ~ 0
-TX0
-Text Label 2200 5950 2    39   ~ 0
-FW_RST
-Text Label 2200 6550 2    39   ~ 0
-GPIO18
-Text Label 2200 6650 2    39   ~ 0
-GPIO19
-Text Label 2200 6750 2    39   ~ 0
-GPIO4
-Text Label 2200 6850 2    39   ~ 0
 GPIO5
-Wire Wire Line
-	2200 5950 1900 5950
-Wire Wire Line
-	1900 5850 2200 5850
 Wire Wire Line
 	2200 5750 1900 5750
@@
 	1150 6750 900  6750
 Wire Wire Line
-	2200 6550 1900 6550
-Wire Wire Line
-	1900 6650 2200 6650
-Wire Wire Line
-	2200 6750 1900 6750
-Wire Wire Line
-	1900 6850 2200 6850
+	2200 5950 1900 5950
+Wire Wire Line
+	1900 6050 2200 6050
+Wire Wire Line
+	2200 6150 1900 6150
+Wire Wire Line
+	1900 6250 2200 6250
 Wire Wire Line
 	6050 5400 5750 5400
@@
 	1    0    0    -1
 $EndComp
-$Comp
-L CONN_01X16 P2
-U 1 1 57EC6E95
-P 1700 6100
-F 0 "P2" H 1700 6950 50  0000 C CNN
-F 1 "CONN_01X16" V 1800 6100 50  0000 C CNN
-F 2 "Pin_Headers:Pin_Header_Straight_1x16" H 1700 6100 50  0001 C CNN
-F 3 "" H 1700 6100 50  0000 C CNN
-	1    1700 6100
+Wire Notes Line
+	2600 6950 750  6950
+Wire Notes Line
+	2600 4950 2600 6950
+Wire Notes Line
+	750  6950 750  4950
+$Comp
+L +5V #PWR0112
+U 1 1 57EC78AB
+P 2400 6250
+F 0 "#PWR0112" H 2400 6100 50  0001 C CNN
+F 1 "+5V" H 2400 6390 50  0000 C CNN
+F 2 "" H 2400 6250 50  0000 C CNN
+F 3 "" H 2400 6250 50  0000 C CNN
+	1    2400 6250
+	1    0    0    -1
+$EndComp
+Wire Wire Line
+	2400 6250 2400 6350
+Wire Wire Line
+	2400 6350 1900 6350
+$Comp
+L CONN_01X11 P2
+U 1 1 57EC8677
+P 1700 5850
+F 0 "P2" H 1700 6450 50  0000 C CNN
+F 1 "CONN_01X11" V 1800 5850 50  0000 C CNN
+F 2 "Pin_Headers:Pin_Header_Straight_1x11" H 1700 5850 50  0001 C CNN
+F 3 "" H 1700 5850 50  0000 C CNN
+	1    1700 5850
 	-1   0    0    -1
 $EndComp
-Wire Notes Line
-	2600 6950 750  6950
-Wire Notes Line
-	2600 4950 2600 6950
-Wire Notes Line
-	750  6950 750  4950
 $EndSCHEMATC
